Commit message: task1

File: 2_wheeledrobot_ws/src/robot_2w_description/urdf/robot_2w_links/base.urdf.xacro (robot description, xacro)
@@ -4,5 +4,5 @@
     <link name="${prefix}base_link">
       <visual>
-        <origin xyz="0 0 0" rpy="0 0 0"/>
+        <origin xyz="0 0 -0.025" rpy="0 0 ${pi/2}"/>
         <geometry>
           <mesh filename="package://robot_2w_description/urdf/meshes/robot2w_chassis.stl" scale="0.0005 0.0005 0.0005"/>

File: 2_wheeledrobot_ws/src/robot_2w_description/urdf/robot_2w_links/caster.urdf.xacro (robot description, xacro)
@@ -5,5 +5,5 @@
     <link name="${prefix}caster_link">
       <visual>
-        <origin xyz="0 0 0" rpy="0 0 0"/>
+        <origin xyz="0 0 0" rpy="${pi/2} 0 0"/>
         <geometry>
             <sphere radius="${caster_wheel_radius}"/>
@@ -30,6 +30,6 @@
       <parent link="${prefix}${parent}" />
       <child link="${prefix}caster_link" />
-      <origin xyz="0.0 0.0 0.0" />
-      <axis xyz="0 0 0" />
+      <origin xyz="0.22 0.0 -0.064" />
+      <axis xyz="0 1 0" />
     </joint>
   </xacro:macro>

File: 2_wheeledrobot_ws/src/robot_2w_description/urdf/robot_2w_links/imu.urdf.xacro (robot description, xacro)
@@ -27,5 +27,5 @@
         <parent link="${prefix}${parent}" />
         <child link="${prefix}imu_link" />
-        <origin xyz="0.0 0.0 0.0" />
+        <origin xyz="-0.02 0 0.01" />
     </joint>
   </xacro:macro>

File: 2_wheeledrobot_ws/src/robot_2w_description/urdf/robot_2w_links/ultrasonic.urdf.xacro (robot description, xacro)
@@ -5,5 +5,5 @@
     <link name="${prefix}ultrasonic_sensor_link" >
       <visual>
-        <origin xyz="0 0 0" rpy="0 0 0"/>
+        <origin xyz="-${ultrasonic_cylinder_length/2.0} 0 0" rpy="0 ${pi/2} 0"/>
         <geometry>
           <cylinder length="${ultrasonic_cylinder_length}" radius="${ultrasonic_cylinder_radius}"/>
@@ -12,5 +12,5 @@
       </visual>
       <collision>
-        <origin xyz="-${ultrasonic_cylinder_length/2.0} 0 0" rpy="0 0 0"/>
+        <origin xyz="-${ultrasonic_cylinder_length/2.0} 0 0" rpy="0 ${pi/2} 0"/>
         <geometry>
           <cylinder length="${ultrasonic_cylinder_length}" radius="${ultrasonic_cylinder_radius}"/>
@@ -23,5 +23,5 @@
       <parent link="${prefix}${parent}"/>
       <child link="${prefix}ultrasonic_sensor_link"/>
-      <origin xyz="0.0 0.0 0.0" rpy="0 0 0"/>
+      <origin xyz="-0.263 0.0 0.0" rpy="0 0 0"/>
     </joint>
     <!-- Gazebo Color -->

File: 2_wheeledrobot_ws/src/robot_2w_description/urdf/robot_2w_links/wheel.urdf.xacro (robot description, xacro)
@@ -6,5 +6,5 @@
     <link name="${prefix}${side}_wheel_link">
       <visual>
-        <origin xyz="0 0 0" rpy="0 0 0"/>
+        <origin xyz="0 0 0" rpy="${pi/2} 0 0"/>
         <geometry>
           <cylinder length="${wheel_length}" radius="${wheel_radius}"/>
@@ -31,5 +31,5 @@
         <parent link="${prefix}${parent}" />
         <child link="${prefix}${side}_wheel_link" />
-        <origin xyz="0.0 0.0 0.0" />
+        <origin xyz="-0.02 ${flip*wheel_distance/2.0} -0.045" />
         <axis xyz="0 1 0" />
     </joint>
