Commit message: change

File: 2_wheeledrobot_ws/src/robot_2w_description/urdf/robot_2w_links/ultrasonic.urdf.xacro (robot description, xacro)
@@ -23,5 +23,5 @@
       <parent link="${prefix}${parent}"/>
       <child link="${prefix}ultrasonic_sensor_link"/>
-      <origin xyz="-0.263 0.0 0.0" rpy="0 0 0"/>
+      <origin xyz="0.263 0.0 0.0" rpy="0 0 0"/>
     </joint>
     <!-- Gazebo Color -->
